Commit message: Update ros_shuttle.urdf.xacro

File: my_robot_description/urdf/ros_shuttle.urdf.xacro (robot description, xacro)
@@ -198,39 +198,15 @@
     <plugin>gz_ros2_control/GazeboSimSystem</plugin>
   </hardware>
-  <joint name="wheel_x1_joint">
-    <command_interface name="velocity"/>
-    <state_interface name="velocity"/>
-  </joint>
-  <joint name="wheel_x2_joint">
-    <command_interface name="velocity"/>
-    <state_interface name="velocity"/>
-  </joint>
-  <joint name="wheel_x3_joint">
-    <command_interface name="velocity"/>
-    <state_interface name="velocity"/>
-  </joint>
-  <joint name="wheel_x4_joint">
-    <command_interface name="velocity"/>
-    <state_interface name="velocity"/>
-  </joint>
-  <joint name="wheel_y1_joint">
-    <command_interface name="velocity"/>
-    <state_interface name="velocity"/>
-  </joint>
-  <joint name="wheel_y2_joint">
-    <command_interface name="velocity"/>
-    <state_interface name="velocity"/>
-  </joint>
-  <joint name="wheel_y3_joint">
-    <command_interface name="velocity"/>
-    <state_interface name="velocity"/>
-  </joint>
-  <joint name="wheel_y4_joint">
-    <command_interface name="velocity"/>
-    <state_interface name="velocity"/>
-  </joint>
+  <joint name="wheel_x1_joint"><command_interface name="velocity"/><state_interface name="velocity"/></joint>
+  <joint name="wheel_x2_joint"><command_interface name="velocity"/><state_interface name="velocity"/></joint>
+  <joint name="wheel_x3_joint"><command_interface name="velocity"/><state_interface name="velocity"/></joint>
+  <joint name="wheel_x4_joint"><command_interface name="velocity"/><state_interface name="velocity"/></joint>
+  <joint name="wheel_y1_joint"><command_interface name="velocity"/><state_interface name="velocity"/></joint>
+  <joint name="wheel_y2_joint"><command_interface name="velocity"/><state_interface name="velocity"/></joint>
+  <joint name="wheel_y3_joint"><command_interface name="velocity"/><state_interface name="velocity"/></joint>
+  <joint name="wheel_y4_joint"><command_interface name="velocity"/><state_interface name="velocity"/></joint>
 </ros2_control>
 <gazebo>
-  <plugin filename="libgz_ros2_control-system.so" name="gz_ros2_control::GazeboSimROS2ControlPlugin">
+  <plugin filename="gz_ros2_control-system" name="gz_ros2_control::GazeboSimROS2ControlPlugin">
     <parameters>$(find my_robot_description)/config/controllers.yaml</parameters>
   </plugin>
